Commit message: Clean packages

File: fanuc_better_model/LRMate-200iD.urdf (robot description, URDF)
Before this commit: robot LRMate-200iD, 8 links, 7 joints
Links:
- link Base: geometry collision mesh filename=package://fanuc_better_model/meshes/Base.STL; visual mesh filename=package://fanuc_better_model/meshes/Base.STL
- link J1: geometry collision mesh filename=package://fanuc_better_model/meshes/J1.STL; visual mesh filename=package://fanuc_better_model/meshes/J1.STL
- link J2: geometry collision mesh filename=package://fanuc_better_model/meshes/J2.STL; visual mesh filename=package://fanuc_better_model/meshes/J2.STL
- link J3: geometry collision mesh filename=package://fanuc_better_model/meshes/J3.STL; visual mesh filename=package://fanuc_better_model/meshes/J3.STL
- link J4: geometry collision mesh filename=package://fanuc_better_model/meshes/J4.STL; visual mesh filename=package://fanuc_better_model/meshes/J4.STL
- link J5: geometry collision mesh filename=package://fanuc_better_model/meshes/J5.STL; visual mesh filename=package://fanuc_better_model/meshes/J5.STL
- link J6: geometry collision mesh filename=package://fanuc_better_model/meshes/J6.STL; visual mesh filename=package://fanuc_better_model/meshes/J6.STL
